Commit message: initial gazebo simulation running

File: description/rpibot.urdf.xacro (robot description, xacro)
@@ -2,3 +2,4 @@
 <robot xmlns:xacro="http://www.ros.org.wiki.xacro" name="rpibot">
     <xacro:include filename="rpibot_core.xacro"/>
+    <xacro:include filename="gazebo_control.xacro"/>
 </robot>

File: description/rpibot_core.xacro (robot description, xacro)
@@ -62,4 +62,7 @@
         </xacro:inertial_box>
     </link>
+    <gazebo reference="chassis">
+        <material>Gazebo/White</material>
+    </gazebo>
     <!-- LEFT WHEEL LINK -->
     <joint name="left_wheel_joint" type="continuous">
@@ -85,4 +88,7 @@
         </xacro:inertial_cylinder>
     </link>
+    <gazebo reference="left_wheel">
+        <material>Gazebo/Grey</material>
+    </gazebo>
     <!-- RIGHT WHEEL LINK -->
     <joint name="right_wheel_joint" type="continuous">
@@ -108,4 +114,7 @@
         </xacro:inertial_cylinder>
     </link>
+    <gazebo reference="right_wheel">
+        <material>Gazebo/Grey</material>
+    </gazebo>
     <!-- FRONT LEFT CASTER LINK -->
     <joint name="fl_caster_joint" type="fixed">
@@ -143,4 +152,9 @@
         </xacro:inertial_box>
     </link>
+    <gazebo reference="fl_caster">
+        <material>Gazebo/Grey</material>
+        <mu1 value="0.001"/>
+        <mu2 value="0.001"/>
+    </gazebo>
     <!-- FRONT RIGHT CASTER LINK -->
     <joint name="fr_caster_joint" type="fixed">
@@ -178,4 +192,9 @@
         </xacro:inertial_box>
     </link>
+    <gazebo reference="fr_caster">
+        <material>Gazebo/Grey</material>
+        <mu1 value="0.001"/>
+        <mu2 value="0.001"/>
+    </gazebo>
     <!-- BACK LEFT CASTER LINK -->
     <joint name="bl_caster_joint" type="fixed">
@@ -213,4 +232,9 @@
         </xacro:inertial_box>
     </link>
+    <gazebo reference="bl_caster">
+        <material>Gazebo/Grey</material>
+        <mu1 value="0.001"/>
+        <mu2 value="0.001"/>
+    </gazebo>
     <!-- BACK RIGHT CASTER LINK -->
     <joint name="br_caster_joint" type="fixed">
@@ -248,3 +272,8 @@
         </xacro:inertial_box>
     </link>
+    <gazebo reference="br_caster">
+        <material>Gazebo/Grey</material>
+        <mu1 value="0.001"/>
+        <mu2 value="0.001"/>
+    </gazebo>
 </robot>
