Commit message: latest changes

File: description/gazebo_control.xacro (robot description, xacro)
@@ -9,12 +9,13 @@
             <wheel_radius>0.035</wheel_radius>
             <!-- Limits-->
-             <max_torque>200</max_torque>
-             <max_acceleration>10.0</max_acceleration>
+             <max_linear_acceleration>6.0</max_linear_acceleration>
             <!-- Output-->
             <frame_id>odom</frame_id>
             <child_frame_id>base_link</child_frame_id>
+            <!-- Topics-->
             <topic>cmd_vel</topic>
             <tf_topic>tf</tf_topic>
             <odom_topic>odom</odom_topic>
+            <odom_publisher_frequency>30</odom_publisher_frequency>
         </plugin>
         <plugin filename="gz-sim-joint-state-publisher-system" name="gz::sim::systems::JointStatePublisher">

File: description/rpibot.urdf.xacro (robot description, xacro)
@@ -3,3 +3,4 @@
     <xacro:include filename="rpibot_core.xacro"/>
     <xacro:include filename="gazebo_control.xacro"/>
+    <xacro:include filename="rplidar.xacro"/>
 </robot>

File: description/rpibot_colors.xacro (robot description, xacro)
@@ -16,3 +16,6 @@
         <color rgba="0.5 0.5 0.5 1"/>
     </material>
+    <material name="red">
+        <color rgba="1 0 0 1"/>
+    </material>
 </robot>

File: description/rpibot_core.xacro (robot description, xacro)
@@ -10,11 +10,10 @@
     <xacro:property name="wheel_base" value="0.150"/>
     <!-- BASE LINK -->
-    <link name="base_link">
-    </link>
+    <link name="base_link"></link>
     <!-- CHASSIS LINK -->
     <joint name="chassis_joint" type="fixed">
         <parent link ="base_link"/>
         <child link="chassis"/>
-        <origin xyz="-${robot_length/2} 0 0.012"/>
+        <origin xyz="-${robot_length/2} 0 ${0.012 - wheel_radius}"/>
     </joint>
     <link name="chassis">
@@ -64,4 +63,6 @@
     <gazebo reference="chassis">
         <material>Gazebo/White</material>
+        <mu1 value="0.001"/>
+        <mu2 value="0.001"/>
     </gazebo>
     <!-- LEFT WHEEL LINK -->
@@ -69,5 +70,5 @@
         <parent link ="base_link"/>
         <child link="left_wheel"/>
-        <origin xyz="0 ${wheel_base/2} ${wheel_radius}" rpy="-${pi/2} 0 0"/>
+        <origin xyz="0 ${wheel_base/2} 0" rpy="-${pi/2} 0 0"/>
         <axis xyz="0 0 1"/>
     </joint>
@@ -95,5 +96,5 @@
         <parent link ="base_link"/>
         <child link="right_wheel"/>
-        <origin xyz="0 -${wheel_base/2} ${wheel_radius}" rpy="${pi/2} 0 0"/>
+        <origin xyz="0 -${wheel_base/2} 0" rpy="${pi/2} 0 0"/>
         <axis xyz="0 0 -1"/>
     </joint>
