Commit message: urdf creation for gazebo

File: description/rpibot_core.xacro (robot description, xacro)
@@ -3,8 +3,4 @@
     <xacro:include filename="rpibot_colors.xacro"/>
     <xacro:include filename="inertial_macros.xacro"/>
-    <!-- BASE LINK -->
-    <link name="base_link">
-    </link>
-    <!-- CHASSIS LINK -->
     <xacro:property name="robot_length" value="0.250"/>
     <xacro:property name="robot_width" value="0.190"/>
@@ -13,8 +9,12 @@
     <xacro:property name="wheel_thickness" value="0.020"/>
     <xacro:property name="wheel_base" value="0.150"/>
+    <!-- BASE LINK -->
+    <link name="base_link">
+    </link>
+    <!-- CHASSIS LINK -->
     <joint name="chassis_joint" type="fixed">
         <parent link ="base_link"/>
         <child link="chassis"/>
-        <origin xyz="-${robot_length/2} 0 -.023"/>
+        <origin xyz="-${robot_length/2} 0 0.012"/>
     </joint>
     <link name="chassis">
@@ -66,5 +66,5 @@
         <parent link ="base_link"/>
         <child link="left_wheel"/>
-        <origin xyz="0 ${wheel_base/2} 0" rpy="-${pi/2} 0 0"/>
+        <origin xyz="0 ${wheel_base/2} ${wheel_radius}" rpy="-${pi/2} 0 0"/>
         <axis xyz="0 0 1"/>
     </joint>
@@ -89,5 +89,5 @@
         <parent link ="base_link"/>
         <child link="right_wheel"/>
-        <origin xyz="0 -${wheel_base/2} 0" rpy="${pi/2} 0 0"/>
+        <origin xyz="0 -${wheel_base/2} ${wheel_radius}" rpy="${pi/2} 0 0"/>
         <axis xyz="0 0 -1"/>
     </joint>

Commit message: Update urdf
Removed gazebo parameters for various links and added new parameters with updated friction values.

File: description/rpibot_core.xacro (robot description, xacro)
@@ -61,9 +61,4 @@
         </xacro:inertial_box>
     </link>
-    <gazebo reference="chassis">
-        <material>Gazebo/White</material>
-        <mu1 value="0.001"/>
-        <mu2 value="0.001"/>
-    </gazebo>
     <!-- LEFT WHEEL LINK -->
     <joint name="left_wheel_joint" type="continuous">
@@ -89,7 +84,4 @@
         </xacro:inertial_cylinder>
     </link>
-    <gazebo reference="left_wheel">
-        <material>Gazebo/Grey</material>
-    </gazebo>
     <!-- RIGHT WHEEL LINK -->
     <joint name="right_wheel_joint" type="continuous">
@@ -115,7 +107,4 @@
         </xacro:inertial_cylinder>
     </link>
-    <gazebo reference="right_wheel">
-        <material>Gazebo/Grey</material>
-    </gazebo>
     <!-- FRONT LEFT CASTER LINK -->
     <joint name="fl_caster_joint" type="fixed">
@@ -153,9 +142,4 @@
         </xacro:inertial_box>
     </link>
-    <gazebo reference="fl_caster">
-        <material>Gazebo/Grey</material>
-        <mu1 value="0.001"/>
-        <mu2 value="0.001"/>
-    </gazebo>
     <!-- FRONT RIGHT CASTER LINK -->
     <joint name="fr_caster_joint" type="fixed">
@@ -163,5 +147,5 @@
         <child link="fr_caster"/>
         <origin xyz="0.225 -0.03 -0.007"/>
-    </joint>3
+    </joint>
     <link name="fr_caster">
         <visual>
@@ -193,9 +177,4 @@
         </xacro:inertial_box>
     </link>
-    <gazebo reference="fr_caster">
-        <material>Gazebo/Grey</material>
-        <mu1 value="0.001"/>
-        <mu2 value="0.001"/>
-    </gazebo>
     <!-- BACK LEFT CASTER LINK -->
     <joint name="bl_caster_joint" type="fixed">
@@ -233,9 +212,4 @@
         </xacro:inertial_box>
     </link>
-    <gazebo reference="bl_caster">
-        <material>Gazebo/Grey</material>
-        <mu1 value="0.001"/>
-        <mu2 value="0.001"/>
-    </gazebo>
     <!-- BACK RIGHT CASTER LINK -->
     <joint name="br_caster_joint" type="fixed">
@@ -273,8 +247,32 @@
         </xacro:inertial_box>
     </link>
+    <!-- Gazebo Parameters -->
+    <gazebo reference="left_wheel">
+        <mu1>1.0</mu1>
+        <mu2>1.0</mu2>
+    </gazebo>
+    <gazebo reference="right_wheel">
+        <mu1>1.0</mu1>
+        <mu2>1.0</mu2>
+    </gazebo>
+    <gazebo reference="fl_caster">
+        <mu1>0.000001</mu1>
+        <mu2>0.000001</mu2>
+    </gazebo>
+    <gazebo reference="fr_caster">
+        <mu1>0.000001</mu1>
+        <mu2>0.000001</mu2>
+    </gazebo>
+    <gazebo reference="bl_caster">
+        <mu1>0.000001</mu1>
+        <mu2>0.000001</mu2>
+    </gazebo>
     <gazebo reference="br_caster">
-        <material>Gazebo/Grey</material>
-        <mu1 value="0.001"/>
-        <mu2 value="0.001"/>
+        <mu1>0.000001</mu1>
+        <mu2>0.000001</mu2>
+    </gazebo>
+    <gazebo reference="base_link">
+        <mu1>1.0</mu1>
+        <mu2>1.0</mu2>
     </gazebo>
 </robot>
