Commit message: updated robot urdf

File: description/robot_description.urdf (robot description, URDF)
Before this commit: robot rpibot, 9 links, 8 joints
Links:
- removed link base_link
- removed link lidar_link
- added link laser_frame, mass 0.14191; collision mesh filename=file:///home/steph/dev_ws/src/rpibot/meshes/laser_frame.STL; visual mesh filename=file:///home/steph/dev_ws/src/rpibot/meshes/laser_frame.STL
- link bl_caster_link: mass 0.00185582478601394 -> 0.0018558; geometry collision mesh filename=file:///home/steph/dev_ws/src/rpibot/meshes/bl_caster_link.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; visual mesh filename=file:///home/steph/dev_ws/src/rpibot/meshes/bl_caster_link.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
- link br_caster_link: mass 0.00185582478601394 -> 0.0018558; geometry collision mesh filename=file:///home/steph/dev_ws/src/rpibot/meshes/br_caster_link.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; visual mesh filename=file:///home/steph/dev_ws/src/rpibot/meshes/br_caster_link.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
- link chassis_link: mass 0.820453668355261 -> 0.82316; geometry collision mesh filename=file:///home/steph/dev_ws/src/rpibot/meshes/chassis_link.STL; visual mesh filename=file:///home/steph/dev_ws/src/rpibot/meshes/chassis_link.STL
- link fl_caster_link: mass 0.00185582478601395 -> 0.0018558; geometry collision mesh filename=file:///home/steph/dev_ws/src/rpibot/meshes/fl_caster_link.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; visual mesh filename=file:///home/steph/dev_ws/src/rpibot/meshes/fl_caster_link.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
- link fr_caster_link: mass 0.00185582478601394 -> 0.0018558; geometry collision mesh filename=file:///home/steph/dev_ws/src/rpibot/meshes/fr_caster_link.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; visual mesh filename=file:///home/steph/dev_ws/src/rpibot/meshes/fr_caster_link.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
- link left_wheel_link: mass 0.0472961083388951 -> 0.047296; geometry collision mesh filename=file:///home/steph/dev_ws/src/rpibot/meshes/left_wheel_link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; visual mesh filename=file:///home/steph/dev_ws/src/rpibot/meshes/left_wheel_link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
- link right_wheel_link: mass 0.0472961083388952 -> 0.047296; geometry collision mesh filename=file:///home/steph/dev_ws/src/rpibot/meshes/right_wheel_lin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; visual mesh filename=file:///home/steph/dev_ws/src/rpibot/meshes/right_wheel_lin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
Joints:
- removed joint chassis_joint
- removed joint lidar_joint
- added joint laser_joint: type fixed, parent chassis_link, child laser_frame, origin xyz=0.043063 0 0.0986 rpy=0 0 0, axis 0 0 0
- joint bl_caster_joint: origin xyz=-0.0999373906923307 0.0500000000000001 -0.0140000000000002 rpy=0 0 0 -> xyz=-0.099937 0.05 -0.014 rpy=0 0 0
- joint fr_caster_joint: origin xyz=0.100062609307669 -0.05 -0.0140000000000002 rpy=0 0 0 -> xyz=0.10006 -0.05 -0.014 rpy=0 0 0
- joint left_wheel_joint: axis 0 0 -1 -> 0 0 1

File: description/robot_description.urdf.xacro (robot description, xacro)
@@ -3,22 +3,27 @@
      Commit Version: 1.6.0-4-g7f85cfe  Build Version: 1.6.7995.38578
      For more information, please see http://wiki.ros.org/sw_urdf_exporter -->
-<robot xmlns:xacro="http://www.ros.org/wiki/xacro" >
-  <link name="base_link">
-  </link>
+<robot
+  name="Simplified Assembly">
+  <link name="base_link"></link>
+  <joint name="chassis_joint" type="fixed">
+        <parent link ="base_link"/>
+        <child link="chassis_link"/>
+        <origin xyz="0 0 -0.0155"/>
+    </joint>
   <link
     name="chassis_link">
     <inertial>
       <origin
-        xyz="1.89291834099631E-05 -5.21505606329551E-17 0.0261554583179408"
-        rpy="0 0 0" />
-      <mass
-        value="0.820453668355261" />
-      <inertia
-        ixx="0.00343745597720794"
-        ixy="-1.33118464296835E-18"
-        ixz="3.3239094876414E-08"
-        iyy="0.00376355614223957"
-        iyz="-3.64969624858544E-20"
-        izz="0.00716840725205158" />
+        xyz="0.00018354 -4.7554E-17 0.026293"
+        rpy="0 0 0" />
+      <mass
+        value="0.82316" />
+      <inertia
+        ixx="0.0034397"
+        ixy="-1.2451E-18"
+        ixz="-1.9509E-06"
+        iyy="0.0037743"
+        iyz="3.903E-21"
+        izz="0.0071801" />
     </inertial>
     <visual>
@@ -33,5 +38,5 @@
         name="">
         <color
-          rgba="0.894117647058823 0.894117647058823 0.894117647058823 1" />
+          rgba="0.11373 0.11373 0.11373 1" />
       </material>
     </visual>
@@ -46,25 +51,19 @@
     </collision>
   </link>
-  <joint name="chassis_joint" type="fixed">
-    <parent link = "base_link"/>
-    <child link = "chassis_link"/>
-    <origin
-      xyz="0 0 -0.0155"/>
-  </joint>
   <link
     name="left_wheel_link">
     <inertial>
       <origin
-        xyz="1.16035451535532E-18 6.93889390390723E-18 -0.00268837094059923"
-        rpy="0 0 0" />
-      <mass
-        value="0.0472961083388951" />
-      <inertia
-        ixx="2.11909458848976E-05"
-        ixy="-2.64101464026675E-24"
-        ixz="-1.58457368331281E-21"
-        iyy="2.11909458848976E-05"
-        iyz="-4.44100545083484E-21"
-        izz="3.991342842481E-05" />
+        xyz="1.8238E-18 6.9389E-18 -0.0026884"
+        rpy="0 0 0" />
+      <mass
+        value="0.047296" />
+      <inertia
+        ixx="2.1191E-05"
+        ixy="9.6271E-24"
+        ixz="-1.6895E-21"
+        iyy="2.1191E-05"
+        iyz="-4.4638E-21"
+        izz="3.9913E-05" />
     </inertial>
     <visual>
@@ -79,5 +78,5 @@
         name="">
         <color
-          rgba="0.752941176470588 0.752941176470588 0.752941176470588 1" />
+          rgba="0.75294 0.75294 0.75294 1" />
       </material>
     </visual>
@@ -112,15 +111,15 @@
     <inertial>
       <origin
-        xyz="-8.43242183162668E-19 -3.46944695195361E-18 -0.00268837094059922"
-        rpy="0 0 0" />
-      <mass
-        value="0.0472961083388952" />
-      <inertia
-        ixx="2.11909458848976E-05"
-        ixy="2.43960739247573E-25"
-        ixz="-2.70461141026291E-21"
-        iyy="2.11909458848976E-05"
-        iyz="4.48416145737291E-21"
-        izz="3.991342842481E-05" />
+        xyz="-6.8682E-19 -6.9389E-18 -0.0026884"
+        rpy="0 0 0" />
+      <mass
+        value="0.047296" />
+      <inertia
+        ixx="2.1191E-05"
+        ixy="3.2915E-24"
+        ixz="-2.665E-21"
+        iyy="2.1191E-05"
+        iyz="4.4967E-21"
+        izz="3.9913E-05" />
     </inertial>
     <visual>
@@ -135,5 +134,5 @@
         name="">
         <color
-          rgba="0.752941176470588 0.752941176470588 0.752941176470588 1" />
+          rgba="0.75294 0.75294 0.75294 1" />
       </material>
     </visual>
@@ -168,37 +167,37 @@
     <inertial>
       <origin
-        xyz="0 3.38181918277552E-34 -0.00900000000000002"
-        rpy="0 0 0" />
-      <mass
-        value="0.069272118011655" />
-      <inertia
-        ixx="2.3084933327384E-05"
-        ixy="-6.627262350311E-53"
-        ixz="-7.99343462295646E-38"
-        iyy="2.3084933327384E-05"
-        iyz="4.21678399541948E-38"
-        izz="4.24291722821387E-05" />
-    </inertial>
-    <visual>
-      <origin
-        xyz="0 0 0"
-        rpy="0 0 0" />
-      <geometry>
-        <mesh
-          filename="file:///home/steph/dev_ws/src/rpibot/meshes/lidar_link.STL" />
-      </geometry>
-      <material
-        name="">
-        <color
-          rgba="0.101960784313725 0.101960784313725 0.101960784313725 1" />
-      </material>
-    </visual>
-    <collision>
-      <origin
-        xyz="0 0 0"
-        rpy="0 0 0" />
-      <geometry>
-        <mesh
-          filename="file:///home/steph/dev_ws/src/rpibot/meshes/lidar_link.STL" />
+        xyz="0.005623 0.00037822 -0.010179"
+        rpy="0 0 0" />
+      <mass
+        value="0.14191" />
+      <inertia
+        ixx="4.5116E-05"
+        ixy="-1.0948E-06"
+        ixz="3.8297E-06"
+        iyy="7.0681E-05"
+        iyz="-1.5038E-07"
+        izz="0.00010464" />
+    </inertial>
+    <visual>
+      <origin
+        xyz="0 0 0"
+        rpy="0 0 0" />
+      <geometry>
+        <mesh
+          filename="file:///home/steph/dev_ws/src/rpibot/meshes/laser_frame.STL" />
+      </geometry>
+      <material
+        name="">
+        <color
+          rgba="0.10196 0.10196 0.10196 1" />
+      </material>
+    </visual>
+    <collision>
+      <origin
+        xyz="0 0 0"
+        rpy="0 0 0" />
+      <geometry>
+        <mesh
+          filename="file:///home/steph/dev_ws/src/rpibot/meshes/laser_frame.STL" />
       </geometry>
     </collision>
@@ -208,5 +207,5 @@
     type="fixed">
     <origin
-      xyz="0.0430626093076691 0 0.1076"
+      xyz="0.043063 0 0.0986"
       rpy="0 0 0" />
     <parent
@@ -216,4 +215,7 @@
     <axis
       xyz="0 0 0" />
+    <dynamics
+      damping="1"
+      friction="1" />
   </joint>
   <link
@@ -221,15 +223,15 @@
     <inertial>
       <origin
-        xyz="2.4980018054066E-16 -2.28983498828939E-16 0.00173996480983857"
-        rpy="0 0 0" />
-      <mass
-        value="0.00185582478601394" />
-      <inertia
-        ixx="4.88878926195383E-08"
-        ixy="-8.68097383355364E-24"
-        ixz="-7.56774428886561E-24"
-        iyy="4.88878926195383E-08"
-        iyz="7.26988457651607E-24"
-        izz="8.72776470384957E-08" />
+        xyz="2.3592E-16 -2.2898E-16 0.00174"
+        rpy="0 0 0" />
+      <mass
+        value="0.0018558" />
+      <inertia
+        ixx="4.8888E-08"
+        ixy="-7.7048E-24"
+        ixz="-7.4938E-24"
+        iyy="4.8888E-08"
+        iyz="7.4281E-24"
+        izz="8.7278E-08" />
     </inertial>
     <visual>
@@ -244,5 +246,5 @@
         name="">
         <color
-          rgba="0.894117647058823 0.894117647058823 0.894117647058823 1" />
+          rgba="0.89412 0.89412 0.89412 1" />
       </material>
     </visual>
@@ -261,5 +263,5 @@
     type="fixed">
     <origin
-      xyz="0.100062609307669 -0.05 -0.0140000000000002"
+      xyz="0.10006 -0.05 -0.014"
       rpy="0 0 0" />
     <parent
@@ -277,15 +279,15 @@
     <inertial>
       <origin
-        xyz="-2.35922392732846E-16 2.35922392732846E-16 0.00173996480983857"
-        rpy="0 0 0" />
-      <mass
-        value="0.00185582478601395" />
-      <inertia
-        ixx="4.88878926195383E-08"
-        ixy="-6.4080026359354E-24"
-        ixz="-4.02583502590903E-24"
-        iyy="4.88878926195382E-08"
-        iyz="6.03349241917912E-24"
-        izz="8.72776470384956E-08" />
+        xyz="-2.3592E-16 2.3592E-16 0.00174"
+        rpy="0 0 0" />
+      <mass
+        value="0.0018558" />
+      <inertia
+        ixx="4.8888E-08"
+        ixy="-6.3701E-24"
+        ixz="-4.0635E-24"
+        iyy="4.8888E-08"
+        iyz="6.0709E-24"
+        izz="8.7278E-08" />
     </inertial>
     <visual>
@@ -300,5 +302,5 @@
         name="">
         <color
-          rgba="0.894117647058823 0.894117647058823 0.894117647058823 1" />
+          rgba="0.89412 0.89412 0.89412 1" />
       </material>
     </visual>
@@ -333,15 +335,15 @@
     <inertial>
       <origin
-        xyz="2.08166817117217E-16 -2.42861286636753E-16 0.00173996480983857"
-        rpy="0 0 0" />
-      <mass
-        value="0.00185582478601394" />
-      <inertia
-        ixx="4.88878926195383E-08"
-        ixy="-1.37377911142332E-23"
-        ixz="1.36549320788026E-23"
-        iyy="4.88878926195381E-08"
-        iyz="1.98579367826622E-24"
-        izz="8.72776470384955E-08" />
+        xyz="2.0817E-16 -2.4286E-16 0.00174"
+        rpy="0 0 0" />
+      <mass
+        value="0.0018558" />
+      <inertia
+        ixx="4.8888E-08"
+        ixy="-1.2961E-23"
+        ixz="1.359E-23"
+        iyy="4.8888E-08"
+        iyz="2.209E-24"
+        izz="8.7278E-08" />
     </inertial>
     <visual>
@@ -356,5 +358,5 @@
         name="">
         <color
-          rgba="0.894117647058823 0.894117647058823 0.894117647058823 1" />
+          rgba="0.89412 0.89412 0.89412 1" />
       </material>
     </visual>
@@ -389,15 +391,15 @@
     <inertial>
       <origin
-        xyz="-2.35922392732846E-16 2.28983498828939E-16 0.00173996480983857"
-        rpy="0 0 0" />
-      <mass
-        value="0.00185582478601394" />
-      <inertia
-        ixx="4.88878926195383E-08"
-        ixy="-9.09078648366105E-24"
-        ixz="7.4144911740129E-24"
-        iyy="4.88878926195383E-08"
-        iyz="-7.28785172670583E-24"
-        izz="8.72776470384957E-08" />
+        xyz="-2.3592E-16 2.2898E-16 0.00174"
+        rpy="0 0 0" />
+      <mass
+        value="0.0018558" />
+      <inertia
+        ixx="4.8888E-08"
+        ixy="-8.5126E-24"
+        ixz="7.4999E-24"
+        iyy="4.8888E-08"
+        iyz="-7.4233E-24"
+        izz="8.7278E-08" />
     </inertial>
     <visual>
@@ -412,5 +414,5 @@
         name="">
         <color
-          rgba="0.894117647058823 0.894117647058823 0.894117647058823 1" />
+          rgba="0.89412 0.89412 0.89412 1" />
       </material>
     </visual>
@@ -429,5 +431,5 @@
     type="fixed">
     <origin
-      xyz="-0.0999373906923307 0.0500000000000001 -0.0140000000000002"
+      xyz="-0.099937 0.05 -0.014"
       rpy="0 0 0" />
     <parent
